Commit message: Adding camera at correct position in all robots

File: franka_description/robots/panda/panda.urdf.xacro (robot description, xacro)
@@ -2,7 +2,11 @@
 <robot xmlns:xacro="http://www.ros.org/wiki/xacro" name="panda">
   <xacro:include filename="$(find franka_description)/robots/common/franka_robot.xacro"/>
+  <xacro:include filename="$(find realsense2_description)/urdf/_d435.urdf.xacro"/>
   <xacro:arg name="arm_id" default="panda" />
   <xacro:franka_robot arm_id="$(arg arm_id)"
                       joint_limits="${xacro.load_yaml('$(find franka_description)/robots/panda/joint_limits.yaml')}">
-  </xacro:franka_robot>
+  </xacro:franka_robot>'
+  <xacro:sensor_d435 parent="$(arg arm_id)_link8">
+  	<origin xyz="0.025 -0.025 0.05" rpy="${-pi/4} ${-pi/2} 0" />
+  </xacro:sensor_d435>
 </robot>
