Commit message: Adding Realsense camera to the robot

File: franka_description/robots/common/franka_arm.xacro (robot description, xacro)
@@ -13,4 +13,10 @@
       </joint>
     </xacro:unless>
+    <link name="world"/>
+    <joint name="robot_to_world" type="fixed">
+	  <parent link="world" />
+	  <child link="${arm_id}_link0" />
+	  <origin xyz="0.0 0.0 0.0" rpy="0.0 0.0 0.0" />
+	</joint>
     <xacro:link_with_sc name="link0" gazebo="${gazebo}">
       <self_collision_geometries>

File: franka_description/robots/common/franka_robot.xacro (robot description, xacro)
@@ -4,5 +4,5 @@
     <!-- Name of this panda -->
     <!-- Should a franka_gripper be mounted at the flange?" -->
-    <xacro:arg name="hand" default="false" />
+    <xacro:arg name="hand" default="true" />
     <!-- Positional offset between $(arm_id)_hand -> $(arm_id)_hand_tcp [m]. Only used when hand:=true -->
     <xacro:arg name="tcp_xyz" default="0 0 0.1034" />

File: franka_description/robots/fr3/fr3.urdf.xacro (robot description, xacro)
@@ -2,7 +2,11 @@
 <robot xmlns:xacro="http://www.ros.org/wiki/xacro" name="fr3">
   <xacro:include filename="$(find franka_description)/robots/common/franka_robot.xacro"/>
+  <xacro:include filename="$(find realsense2_description)/urdf/_d435.urdf.xacro"/>
   <xacro:arg name="arm_id" default="fr3" />
   <xacro:franka_robot arm_id="$(arg arm_id)"
                       joint_limits="${xacro.load_yaml('$(find franka_description)/robots/fr3/joint_limits.yaml')}">
   </xacro:franka_robot>
+  <xacro:sensor_d435 parent="$(arg arm_id)_link8">
+  	<origin xyz="0.05 0 0.05" rpy="${-pi/4} ${-pi/2} 0" />
+  </xacro:sensor_d435>
 </robot>

Commit message: removing additional world frame from urdf

File: franka_description/robots/common/franka_arm.xacro (robot description, xacro)
@@ -13,10 +13,4 @@
       </joint>
     </xacro:unless>
-    <link name="world"/>
-    <joint name="robot_to_world" type="fixed">
-	  <parent link="world" />
-	  <child link="${arm_id}_link0" />
-	  <origin xyz="0.0 0.0 0.0" rpy="0.0 0.0 0.0" />
-	</joint>
     <xacro:link_with_sc name="link0" gazebo="${gazebo}">
       <self_collision_geometries>
