Commit message: Changing gazebo and inertial values for moveit visualization

File: franka_description/robots/common/franka_hand.xacro (robot description, xacro)
@@ -106,5 +106,5 @@
       <axis xyz="0 1 0" />
       <limit effort="100" lower="0.0" upper="0.04" velocity="0.2" />
-      <dynamics damping="0.3" />
+      <dynamics damping="1" />
     </joint>
     <joint name="${arm_id}_finger_joint2" type="prismatic">
@@ -115,5 +115,5 @@
       <limit effort="100" lower="0.0" upper="0.04" velocity="0.2" />
       <mimic joint="${arm_id}_finger_joint1" />
-      <dynamics damping="0.3" />
+      <dynamics damping="1" />
     </joint>
   </xacro:macro>

File: franka_description/robots/common/franka_robot.xacro (robot description, xacro)
@@ -37,5 +37,5 @@
         <child  link="$(arg arm_id)_link0" />
       </joint>
-      <xacro:gazebo-joint joint="${arm_id}_joint1" transmission="hardware_interface/PositionJointInterface" />
+      <!-- <xacro:gazebo-joint joint="${arm_id}_joint1" transmission="hardware_interface/PositionJointInterface" />
       <xacro:gazebo-joint joint="${arm_id}_joint2" transmission="hardware_interface/PositionJointInterface" />
       <xacro:gazebo-joint joint="${arm_id}_joint3" transmission="hardware_interface/PositionJointInterface" />
@@ -50,5 +50,5 @@
       <xacro:gazebo-joint joint="${arm_id}_joint5" transmission="hardware_interface/VelocityJointInterface" />
       <xacro:gazebo-joint joint="${arm_id}_joint6" transmission="hardware_interface/VelocityJointInterface" />
-      <xacro:gazebo-joint joint="${arm_id}_joint7" transmission="hardware_interface/VelocityJointInterface" />
+      <xacro:gazebo-joint joint="${arm_id}_joint7" transmission="hardware_interface/VelocityJointInterface" /> -->
       <xacro:gazebo-joint joint="${arm_id}_joint1" transmission="hardware_interface/EffortJointInterface" />
       <xacro:gazebo-joint joint="${arm_id}_joint2" transmission="hardware_interface/EffortJointInterface" />
@@ -58,9 +58,9 @@
       <xacro:gazebo-joint joint="${arm_id}_joint6" transmission="hardware_interface/EffortJointInterface" />
       <xacro:gazebo-joint joint="${arm_id}_joint7" transmission="hardware_interface/EffortJointInterface" />
-      <xacro:transmission-franka-state arm_id="${arm_id}" />
+      <!-- <xacro:transmission-franka-state arm_id="${arm_id}" />
       <xacro:transmission-franka-model arm_id="${arm_id}"
          root="${arm_id}_joint1"
          tip="${arm_id}_joint8"
-       />
+       /> -->
       <xacro:if value="$(arg hand)">
         <xacro:gazebo-joint joint="${arm_id}_finger_joint1" transmission="hardware_interface/EffortJointInterface" />
@@ -72,8 +72,8 @@
       <gazebo>
         <plugin name="gazebo_ros_control" filename="libgazebo_ros_control.so">
-          <controlPeriod>0.001</controlPeriod>
-          <robotSimType>franka_gazebo/FrankaHWSim</robotSimType>
+          <!-- <controlPeriod>0.001</controlPeriod>
+          <robotSimType>franka_gazebo/FrankaHWSim</robotSimType> -->
         </plugin>
-        <self_collide>true</self_collide>
+        <!-- <self_collide>true</self_collide> -->
       </gazebo>
     </xacro:if>

File: franka_description/robots/common/utils.xacro (robot description, xacro)
@@ -113,5 +113,8 @@
     <gazebo reference="${joint}">
       <!-- Needed for ODE to output external wrenches on joints -->
-      <provideFeedback>true</provideFeedback>
+      <!-- <provideFeedback>true</provideFeedback> -->
+      <mu1>0.2</mu1>
+      <mu2>0.2</mu2>
+      <!-- <gravity>0</gravity> -->
     </gazebo>
     <transmission name="${joint}_transmission">
@@ -122,4 +125,5 @@
       <actuator name="${joint}_motor">
         <hardwareInterface>${transmission}</hardwareInterface>
+        <mechanicalReduction>1</mechanicalReduction>
       </actuator>
     </transmission>

File: franka_description/robots/fr3/fr3.urdf.xacro (robot description, xacro)
@@ -8,5 +8,5 @@
   </xacro:franka_robot>
   <xacro:sensor_d435 parent="$(arg arm_id)_link8">
-  	<origin xyz="0.05 0 0.05" rpy="${-pi/4} ${-pi/2} 0" />
+  	<origin xyz="0.025 -0.025 0.05" rpy="${-pi/4} ${-pi/2} 0" />
   </xacro:sensor_d435>
 </robot>

File: franka_description/robots/panda/panda.urdf.xacro (robot description, xacro)
@@ -6,5 +6,5 @@
   <xacro:franka_robot arm_id="$(arg arm_id)"
                       joint_limits="${xacro.load_yaml('$(find franka_description)/robots/panda/joint_limits.yaml')}">
-  </xacro:franka_robot>'
+  </xacro:franka_robot>
   <xacro:sensor_d435 parent="$(arg arm_id)_link8">
   	<origin xyz="0.025 -0.025 0.05" rpy="${-pi/4} ${-pi/2} 0" />
